File: design.kicad_sch (KiCad schematic)
At the start: 0 parts

Commit message: UPDATE
Parts:
- added C1: 47uF, Capacitor_SMD:C_0805_2012Metric, symbol Device:C_Small
- added C2: 22uF, Capacitor_SMD:C_0805_2012Metric, symbol Device:C_Small
- added D1: 1N5817, Diode_THT:D_T-1_P10.16mm_Horizontal, symbol Device:D_Schottky
- added J1, J2: Conn_02x02_Counter_Clockwise, Connector_PinHeader_2.54mm:PinHeader_2x02_P2.54mm_Vertical, symbol Connector_Generic:Conn_02x02_Counter_Clockwise
- added L1: 47uH, Inductor_SMD:L_Vishay_IFSC-1515AH_4x4x1.8mm, symbol Device:L_Small
- added R1: 0.15, Resistor_SMD:R_0805_2012Metric, symbol Device:R_Small
- added TP1, TP2, TP3, TP4: TestPoint, TestPoint:TestPoint_Pad_D3.0mm, symbol Connector:TestPoint
- added TP5, TP6, TP7, TP8: RCWCTE, Snapeda:RCWCTE_TP420X150, symbol Snapeda:RCWCTE
- added U1: HT77xxBA, Package_TO_SOT_SMD:SOT-23-5, symbol Converter_DCDC_custom:HT77xxBA
Connections:
- new net: C2.1, R1.2
- new net GND: C1.2, C2.2, J1.1 (Pin_1), J1.2 (Pin_2), J2.1 (Pin_1), J2.2 (Pin_2), TP3.1, TP4.1, TP7.1, TP8.1, U1.4 (GND)
- new net LX: D1.2 (A), L1.2, U1.5 (LX)
- new net Vin: C1.1, J1.3 (Pin_3), J1.4 (Pin_4), L1.1, TP1.1, TP5.1
- new net Vout: D1.1 (K), J2.3 (Pin_3), J2.4 (Pin_4), R1.1, TP2.1, TP6.1, U1.1 (CE), U1.2 (OUT)
