File: design.kicad_sch (KiCad schematic)
At the start: 16 parts, among them J1 Conn_02x02_Counter_Clockwise, J2 Conn_02x02_Counter_Clockwise, U1 HT77xxBA

Commit message: update
Parts:
- TP1: value TestPoint -> Vin
- TP2: value TestPoint -> Vout
- TP3, TP4: value TestPoint -> GND
Changed lines of the file:
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@@
   (junction (at 205.74 64.77) (diameter 0) (color 0 0 0 0)
   )
+  (junction (at 147.32 98.425) (diameter 0) (color 0 0 0 0)
+  )
   (junction (at 236.22 64.77) (diameter 0) (color 0 0 0 0)
   )
@@
   (junction (at 133.985 86.36) (diameter 0) (color 0 0 0 0)
   )
+  (junction (at 133.985 71.12) (diameter 0) (color 0 0 0 0)
+  )
   (wire (pts (xy 133.985 71.12) (xy 133.985 86.36))
     (stroke (width 0) (type default) (color 0 0 0 0))
@@
     (stroke (width 0) (type default) (color 0 0 0 0))
   )
-  (wire (pts (xy 147.32 96.52) (xy 147.32 100.33))
+  (wire (pts (xy 147.32 96.52) (xy 147.32 98.425))
     (stroke (width 0) (type default) (color 0 0 0 0))
   )
@@
   )
   (wire (pts (xy 173.99 93.98) (xy 173.99 97.79))
+    (stroke (width 0) (type default) (color 0 0 0 0))
+  )
+  (wire (pts (xy 147.32 98.425) (xy 147.32 100.33))
     (stroke (width 0) (type default) (color 0 0 0 0))
   )
@@
       (effects (font (size 1.27 1.27)) (justify left))
     )
-    (property "Value" "TestPoint" (id 1) (at 214.63 66.0399 90)
+    (property "Value" "GND" (id 1) (at 214.63 66.0399 90)
       (effects (font (size 1.27 1.27)) (justify left))
     )
@@
       (effects (font (size 1.27 1.27)) (justify left))
     )
-    (property "Value" "TestPoint" (id 1) (at 214.63 59.6899 90)
+    (property "Value" "GND" (id 1) (at 214.63 59.6899 90)
       (effects (font (size 1.27 1.27)) (justify left))
     )
@@
     (pin "1")
   )
+  (symbol (lib_id "power:PWR_FLAG") (at 133.985 71.12 0) (unit 1)
+    (in_bom yes) (on_board yes) (fields_autoplaced)
+    (property "Reference" "#FLG0101" (id 0) (at 133.985 69.215 0)
+      (effects (font (size 1.27 1.27)) hide)
+    )
+    (property "Value" "PWR_FLAG" (id 1) (at 133.985 66.04 0))
+    (property "Footprint" "" (id 2) (at 133.985 71.12 0)
+      (effects (font (size 1.27 1.27)) hide)
+    )
+    (property "Datasheet" "~" (id 3) (at 133.985 71.12 0)
+      (effects (font (size 1.27 1.27)) hide)
+    )
+    (pin "1")
+  )
   (symbol (lib_id "Connector_Generic:Conn_02x02_Counter_Clockwise") (at 112.395 133.985 0) (unit 1)
     (in_bom yes) (on_board yes) (fields_autoplaced)
@@
     (pin "2")
   )
+  (symbol (lib_id "power:PWR_FLAG") (at 147.32 98.425 270) (unit 1)
+    (in_bom yes) (on_board yes) (fields_autoplaced)
+    (property "Reference" "#FLG0102" (id 0) (at 149.225 98.425 0)
+      (effects (font (size 1.27 1.27)) hide)
+    )
+    (property "Value" "PWR_FLAG" (id 1) (at 151.13 98.4249 90)
+      (effects (font (size 1.27 1.27)) (justify left))
+    )
+    (property "Footprint" "" (id 2) (at 147.32 98.425 0)
+      (effects (font (size 1.27 1.27)) hide)
+    )
+    (property "Datasheet" "~" (id 3) (at 147.32 98.425 0)
+      (effects (font (size 1.27 1.27)) hide)
+    )
+    (pin "1")
+  )
   (symbol (lib_id "Connector:TestPoint") (at 209.55 45.72 270) (unit 1)
     (in_bom yes) (on_board yes) (fields_autoplaced)
@@
       (effects (font (size 1.27 1.27)) (justify left))
     )
-    (property "Value" "TestPoint" (id 1) (at 214.63 46.9899 90)
+    (property "Value" "Vin" (id 1) (at 214.63 46.9899 90)
       (effects (font (size 1.27 1.27)) (justify left))
     )
@@
       (effects (font (size 1.27 1.27)) (justify left))
     )
-    (property "Value" "TestPoint" (id 1) (at 214.63 53.3399 90)
+    (property "Value" "Vout" (id 1) (at 214.63 53.3399 90)
       (effects (font (size 1.27 1.27)) (justify left))
     )
@@
   )
   (symbol_instances
+    (path "/cc4a2e72-0721-4902-b764-106ec75391d6"
+      (reference "#FLG0101") (unit 1) (value "PWR_FLAG") (footprint "")
+    )
+    (path "/dbd05475-acd6-4d51-86ea-f0383604bcf0"
+      (reference "#FLG0102") (unit 1) (value "PWR_FLAG") (footprint "")
+    )
     (path "/ad2c467b-abc6-4f81-a30b-e2bb852955ec"
       (reference "#PWR0101") (unit 1) (value "GND") (footprint "")
@@
     )
     (path "/e7bfdd8c-d5bb-408b-8430-d56e1595941d"
-      (reference "TP1") (unit 1) (value "TestPoint") (footprint "TestPoint:TestPoint_Pad_D3.0mm")
+      (reference "TP1") (unit 1) (value "Vin") (footprint "TestPoint:TestPoint_Pad_D3.0mm")
     )
     (path "/ff26b8c7-7563-4098-9b5c-7a00d21ba52d"
-      (reference "TP2") (unit 1) (value "TestPoint") (footprint "TestPoint:TestPoint_Pad_D3.0mm")
+      (reference "TP2") (unit 1) (value "Vout") (footprint "TestPoint:TestPoint_Pad_D3.0mm")
     )
     (path "/60bae830-0278-4483-94ac-2d880fc8aacc"
-      (reference "TP3") (unit 1) (value "TestPoint") (footprint "TestPoint:TestPoint_Pad_D3.0mm")
+      (reference "TP3") (unit 1) (value "GND") (footprint "TestPoint:TestPoint_Pad_D3.0mm")
     )
     (path "/32b56400-8125-4c3e-a575-9fb4bdc40cb4"
-      (reference "TP4") (unit 1) (value "TestPoint") (footprint "TestPoint:TestPoint_Pad_D3.0mm")
+      (reference "TP4") (unit 1) (value "GND") (footprint "TestPoint:TestPoint_Pad_D3.0mm")
     )
     (path "/78154ced-3f4c-437c-af78-e8307b7a06a7"
