File: design.kicad_pcb (KiCad board)
At the start: 2 copper layers, 47 x 28 mm, 0 parts

Commit message: UPDATE
Parts:
- added C1: 47uF, Capacitor_SMD:C_0805_2012Metric, F.Cu at (113.5, 112.5)
- added C2: 22uF, Capacitor_SMD:C_0805_2012Metric, F.Cu at (128.0, 116.2)
- added D1: 1N5817, Diode_THT:D_T-1_P10.16mm_Horizontal, F.Cu at (127.6, 121.5)
- added J1: Conn_02x02_Counter_Clockwise, Connector_PinHeader_2.54mm:PinHeader_2x02_P2.54mm_Vertical, F.Cu at (105.7, 111.2)
- added J2: Conn_02x02_Counter_Clockwise, Connector_PinHeader_2.54mm:PinHeader_2x02_P2.54mm_Vertical, F.Cu at (134.0, 115.8)
- added L1: 47uH, Inductor_SMD:L_Vishay_IFSC-1515AH_4x4x1.8mm, F.Cu at (117.5, 115.0)
- added R1: 0.15, Resistor_SMD:R_0805_2012Metric, F.Cu at (126.0, 114.4)
- added TP1: Vin, TestPoint:TestPoint_Pad_D3.0mm, F.Cu at (104.5, 119.0)
- added TP2: Vout, TestPoint:TestPoint_Pad_D3.0mm, F.Cu at (138.5, 113.2)
- added TP3: GND, TestPoint:TestPoint_Pad_D3.0mm, F.Cu at (104.5, 125.0)
- added TP4: GND, TestPoint:TestPoint_Pad_D3.0mm, F.Cu at (138.5, 125.0)
- added TP5: RCWCTE, Snapeda:RCWCTE_TP420X150, F.Cu at (110.8, 119.0)
- added TP6: RCWCTE, Snapeda:RCWCTE_TP420X150, F.Cu at (132.8, 109.8)
- added TP7: RCWCTE, Snapeda:RCWCTE_TP420X150, F.Cu at (110.8, 124.0)
- added TP8: RCWCTE, Snapeda:RCWCTE_TP420X150, F.Cu at (132.8, 119.2)
- added U1: HT77xxBA, Package_TO_SOT_SMD:SOT-23-5, F.Cu at (122.5, 112.5)
Routing:
- net Vout: track 0.00 -> 10.8 mm
- net Net-(C2-Pad1): track 0.00 -> 2.01 mm
- net GND: vias 0 -> 16
- added copper zone on F.Cu, net /LX
- added copper zone on B.Cu, net GND
- added copper zone on F.Cu, net GND
- added copper zone on F.Cu, net Vin
- added copper zone on F.Cu, net Vout
Other:
- board size 47 x 28 mm -> 40 x 20 mm
- board text added: "GND"
- board text added: "Vin"
- board text added: "Vout"

Commit message: update
Other:
- outline, holes or cut-outs redrawn
Changed lines of the file:
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@@
   (gr_line (start 141 115.5) (end 135.5 115.5) (layer "F.SilkS") (width 0.12))
   (gr_line (start 112.5 112.5) (end 110 112.5) (layer "F.SilkS") (width 0.12))
-  (gr_line (start 129.75 114.5) (end 123.5 114.5) (layer "F.SilkS") (width 0.12))
+  (gr_line (start 125 114.5) (end 123.5 114.5) (layer "F.SilkS") (width 0.12))
+  (gr_line (start 129.75 114.5) (end 127.25 114.5) (layer "F.SilkS") (width 0.12))
   (gr_line (start 122.5 108.5) (end 122.5 110.75) (layer "F.SilkS") (width 0.12))
   (gr_line (start 116.5 112.5) (end 114.5 112.5) (layer "F.SilkS") (width 0.12))
-  (gr_line (start 141 108.5) (end 141 115.5) (layer "F.SilkS") (width 0.12))
+  (gr_arc (start 138 108.5) (mid 140.12132 109.37868) (end 141 111.5) (layer "F.SilkS") (width 0.12))
+  (gr_line (start 141 111.5) (end 141 115.5) (layer "F.SilkS") (width 0.12))
   (gr_line (start 102 112.495) (end 102 121.25) (layer "F.SilkS") (width 0.12))
   (gr_line (start 115.25 121.25) (end 115.25 119.5) (layer "F.SilkS") (width 0.12))
-  (gr_line (start 122.5 108.5) (end 141 108.5) (layer "F.SilkS") (width 0.12))
+  (gr_line (start 122.5 108.5) (end 138 108.5) (layer "F.SilkS") (width 0.12))
   (gr_line (start 102 112.495) (end 104 112.495) (layer "F.SilkS") (width 0.12))
   (gr_line (start 115.25 119.5) (end 117.25 117.75) (layer "F.SilkS") (width 0.12))
   (gr_line (start 102 121.25) (end 115.25 121.25) (layer "F.SilkS") (width 0.12))
-  (gr_rect (start 101.5 108) (end 141.5 128) (layer "Edge.Cuts") (width 0.05) (fill none))
+  (gr_arc (start 141.5 125) (mid 140.62132 127.12132) (end 138.5 128) (layer "Edge.Cuts") (width 0.05))
+  (gr_line (start 141.5 111) (end 141.5 125) (layer "Edge.Cuts") (width 0.05))
+  (gr_arc (start 138.5 108) (mid 140.62132 108.87868) (end 141.5 111) (layer "Edge.Cuts") (width 0.05))
+  (gr_arc (start 101.5 111) (mid 102.37868 108.87868) (end 104.5 108) (layer "Edge.Cuts") (width 0.05))
+  (gr_line (start 104.5 108) (end 138.5 108) (layer "Edge.Cuts") (width 0.05))
+  (gr_line (start 101.5 125) (end 101.5 111) (layer "Edge.Cuts") (width 0.05))
+  (gr_arc (start 104.5 128) (mid 102.37868 127.12132) (end 101.5 125) (layer "Edge.Cuts") (width 0.05))
+  (gr_line (start 138.5 128) (end 104.5 128) (layer "Edge.Cuts") (width 0.05))
   (gr_text "<<project_name>>\n<<ID>>\n<<version>>\n<<date>>\n<<hash>>\n<<website_link>>" (at 121.75 115.5) (layer "B.SilkS")
     (effects (font (size 1 1) (thickness 0.15)) (justify mirror))
@@
     (polygon
       (pts
+        (xy 139.735955 109)
+        (xy 140.5 109.75)
+        (xy 141 110.75)
         (xy 141 115.5)
         (xy 135.75 115.5)
@@
         (xy 122.5 114.5)
         (xy 122.5 108.5)
-        (xy 141 108.5)
+        (xy 138.5 108.5)
       )
     )
